Commit message: Update robot.urdf

File: urdf/robot.urdf (robot description, URDF)
Before this commit: robot line_following_robot, 5 links, 4 joints
Joints:
- joint left_front_wheel_joint: origin xyz=-0.15 0.1 0 rpy=0 0 0 -> xyz=0.15 -0.1 0 rpy=0 0 0
- joint left_rear_wheel_joint: origin xyz=0.15 0.1 0 rpy=0 0 0 -> xyz=-0.15 -0.1 0 rpy=0 0 0
- joint right_front_wheel_joint: origin xyz=-0.15 -0.1 0 rpy=0 0 0 -> xyz=-0.15 0.1 0 rpy=0 0 0
- joint right_rear_wheel_joint: origin xyz=0.15 -0.1 0 rpy=0 0 0 -> xyz=-0.15 0.1 0 rpy=0 0 0
